Commit message: fix executing trajectory and general updates pt2

File: src/ur5e_2fg7/urdf/ur5e_2fg7.ros2_control.xacro (robot description, xacro)
@@ -1,68 +1,53 @@
 <?xml version="1.0"?>
 <robot xmlns:xacro="http://www.ros.org/wiki/xacro">
-  <!-- <xacro:macro name="ur5e_2fg7_ros2_control" params="name"> -->
-  <xacro:macro name="IsaacSimSystem" params="name">
-    <ros2_control name="${name}" type="system">
-      <!-- <hardware>
-        <plugin>isaac_ros2_control/IsaacSystem</plugin>
-        <param name="joint_commands_topic">/isaac_joint_commands</param>
-        <param name="joint_states_topic">/isaac_joint_states</param>
-      </hardware> -->
-      <hardware>
-        <plugin>topic_based_ros2_control/TopicBasedSystem</plugin>
-        <param name="joint_commands_topic">/isaac_joint_commands</param>
-        <param name="joint_states_topic">/isaac_joint_states</param>
-      </hardware>
-      <joint name="shoulder_pan_joint">
-        <command_interface name="position"/>
-        <state_interface name="position"/>
-        <state_interface name="velocity"/>
-      </joint>
-      <joint name="shoulder_lift_joint">
-        <command_interface name="position"/>
-        <state_interface name="position"/>
-        <state_interface name="velocity"/>
-      </joint>
-      <joint name="elbow_joint">
-        <command_interface name="position"/>
-        <state_interface name="position"/>
-        <state_interface name="velocity"/>
-      </joint>
-      <joint name="wrist_1_joint">
-        <command_interface name="position"/>
-        <state_interface name="position"/>
-        <state_interface name="velocity"/>
-      </joint>
-      <joint name="wrist_2_joint">
-        <command_interface name="position"/>
-        <state_interface name="position"/>
-        <state_interface name="velocity"/>
-      </joint>
-      <joint name="wrist_3_joint">
-        <command_interface name="position"/>
-        <state_interface name="position"/>
-        <state_interface name="velocity"/>
-      </joint>
-      <joint name="gripper_gripper_joint">
-        <command_interface name="position"/>
-        <command_interface name="effort"/>
-        <state_interface name="position"/>
-        <state_interface name="velocity"/>
-        <state_interface name="effort"/>
-      </joint>
-      <joint name="gripper_right_finger_joint">
-        <command_interface name="position"/>
-        <state_interface name="position"/>
-        <state_interface name="velocity"/>
-      </joint>
-      <!-- <sensor name="wrist_3_joint">
-        <state_interface name="force.x"/>
-        <state_interface name="force.y"/>
-        <state_interface name="force.z"/>
-        <state_interface name="torque.x"/>
-        <state_interface name="torque.y"/>
-        <state_interface name="torque.z"/>
-      </sensor> -->
-    </ros2_control>
-  </xacro:macro>
+<!-- <xacro:macro name="ur5e_2fg7_ros2_control" params="name"> -->
+<xacro:macro name="IsaacSimSystem" params="name">
+<ros2_control name="${name}" type="system">
+<hardware>
+<plugin>mock_components/GenericSystem</plugin>
+</hardware>
+<joint name="shoulder_pan_joint">
+<command_interface name="position"/>
+<state_interface name="position"/>
+<state_interface name="velocity"/>
+</joint>
+<joint name="shoulder_lift_joint">
+<command_interface name="position"/>
+<state_interface name="position"/>
+<state_interface name="velocity"/>
+</joint>
+<joint name="elbow_joint">
+<command_interface name="position"/>
+<state_interface name="position"/>
+<state_interface name="velocity"/>
+</joint>
+<joint name="wrist_1_joint">
+<command_interface name="position"/>
+<state_interface name="position"/>
+<state_interface name="velocity"/>
+</joint>
+<joint name="wrist_2_joint">
+<command_interface name="position"/>
+<state_interface name="position"/>
+<state_interface name="velocity"/>
+</joint>
+<joint name="wrist_3_joint">
+<command_interface name="position"/>
+<state_interface name="position"/>
+<state_interface name="velocity"/>
+</joint>
+<joint name="gripper_gripper_joint">
+<command_interface name="position"/>
+<command_interface name="effort"/>
+<state_interface name="position"/>
+<state_interface name="velocity"/>
+<state_interface name="effort"/>
+</joint>
+<joint name="gripper_right_finger_joint">
+<command_interface name="position"/>
+<state_interface name="position"/>
+<state_interface name="velocity"/>
+</joint>
+</ros2_control>
+</xacro:macro>
 </robot>

File: src/ur5e_2fg7/urdf/ur5e_2fg7_main.urdf.xacro (robot description, xacro)
@@ -2,4 +2,5 @@
 <robot xmlns:xacro="http://wiki.ros.org/xacro" name="ur5e_con_2fg7">
   <xacro:include filename="/opt/ros/humble/share/ur_description/urdf/ur_macro.xacro"/>
+  <xacro:include filename="$(find ur5e_2fg7)/urdf/ur5e_2fg7.ros2_control.xacro"/>
   <xacro:include filename="$(find onrobot_2fg7_description)/urdf/onrobot_2fg7.xacro"/>
   <link name="world"/>
@@ -12,5 +13,6 @@
     physical_parameters_file="/opt/ros/humble/share/ur_description/config/ur5e/physical_parameters.yaml"
     visual_parameters_file="/opt/ros/humble/share/ur_description/config/ur5e/visual_parameters.yaml"
-    initial_positions="${dict(shoulder_pan_joint=0.0,shoulder_lift_joint=-1.57,elbow_joint=1.57,wrist_1_joint=-1.57,wrist_2_joint=-1.57,wrist_3_joint=0.0)}">
+    initial_positions="${dict(shoulder_pan_joint=0.0,shoulder_lift_joint=-1.57,elbow_joint=1.57,wrist_1_joint=-1.57,wrist_2_joint=-1.57,wrist_3_joint=0.0)}"
+    use_fake_hardware="true">
     <origin xyz="0 0 0" rpy="0 0 0"/>
   </xacro:ur_robot>
@@ -18,4 +20,5 @@
     <origin xyz="0 0 0" rpy="0 0 0"/>
   </xacro:onrobot_2fg7>
+  <xacro:IsaacSimSystem name="ur5e_2fg7_system"/>
   <material name="pad_black">
     <color rgba="0.1 0.1 0.1 1.0"/>
